File: hw/as5047_breakout/as5047_breakout.sch (EAGLE design)
At the start: 3 parts

Commit message: Rename AS5147->AS5047 which actually seems to exist
Add a MA700 breakout, which I may or may not need
Parts:
- U$1: DPN (none) -> AS5047D-ATSMCT-ND; MFG (none) -> AMS; MPN (none) -> AS5047D-ATSM
Changed lines of the file:
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@@
 </classes>
 <parts>
-<part name="U$1" library="as5147_breakout" deviceset="AS5147" device=""/>
+<part name="U$1" library="as5147_breakout" deviceset="AS5147" device="">
+<attribute name="DPN" value="AS5047D-ATSMCT-ND"/>
+<attribute name="MFG" value="AMS"/>
+<attribute name="MPN" value="AS5047D-ATSM"/>
+</part>
 <part name="C1" library="rcl" deviceset="C-US" device="C0603" value="0.1uF"/>
 <part name="GND1" library="supply1" deviceset="GND" device=""/>
@@
 </plain>
 <instances>
-<instance part="U$1" gate="G$1" x="63.5" y="45.72"/>
+<instance part="U$1" gate="G$1" x="63.5" y="45.72">
+<attribute name="DPN" x="63.5" y="45.72" size="1.778" layer="96" display="off"/>
+<attribute name="MFG" x="63.5" y="45.72" size="1.778" layer="96" display="off"/>
+<attribute name="MPN" x="63.5" y="45.72" size="1.778" layer="96" display="off"/>
+</instance>
 <instance part="C1" gate="G$1" x="27.94" y="38.1"/>
 <instance part="GND1" gate="1" x="43.18" y="22.86"/>
