File: hw/precharge/precharge.sch (EAGLE design)
At the start: 32 parts, among them Q1 TPH1R204PL, Q2 TPH1R204PL, U1 ZXTR2012Z, U2 LP2985SOT-23-5, U3 ATTINY44A-SSU, U4 MIC4416, U5 MIC4416

Commit message: Continued iteration on precharge board
Parts:
- added R8, R9: 100k 1%, mfpassives:RESISTOR_0603
- C3: MF (none) -> KEMET; MPN (none) -> C0603C225K8PACTU
- C4, C5, C6: HOUSEPART (none) -> 1; MPN (none) -> MF-CAP-0603-0.1uF
- D1, D2: HOUSEPART (none) -> 1; MPN (none) -> MF-LED-0603-RED
- JP1: POPULATE (none) -> 0
- R1, R2: HOUSEPART (none) -> 1; MPN (none) -> MF-RES-0603-220
- R3, R5: MF (none) -> VISHAY; MPN (none) -> CRCW0603100KFKEA
- R4, R6: MF (none) -> PANASONIC; MPN (none) -> ERT-J1VG103FA
Connections:
- net FET_MAIN: now also R9.P$2
- net FET_PRECHARGE: now also R8.P$2
- net GND: now also R8.P$1, R9.P$1

Commit message: Updated pre-charge, now named "power distribution"
Nominally everything but auto-route
Parts:
- removed JP1: (no value), pinhead:PINHD-2X3
- removed V+, V+OUT, V-, V-OUT: PAD12AWG_PAD, controller:PAD12AWG_PAD
- added C10, C11, C12, C13: 0.1uF, mfpassives:CAPACITOR_NP_0402
- added C14: 1uF, mfpassives:CAPACITOR_NP_0402
- added C15, C7: 10uF 35V, mfpassives:CAPACITOR_NP_1206
- added C8, C9: 1uF 50V, mfpassives:CAPACITOR_NP_0603
- added CAN1, CAN2: JST-PH3SMT_VERT, precharge:JST-PH3SMT_VERT
- added D12, D3V3, DG: PAD24AWG_PAD, precharge:PAD24AWG_PAD
- added J1: JST-ZH6SMT_VERT, precharge:JST-ZH6SMT_VERT
- added J2: JST-PH4SMT_VERT, precharge:JST-PH4SMT_VERT
- added L1: 33uH, mfpassives:INDUCTOR_1210
- added P1, P2, P3, P4, P5, P6: XT30P, precharge:XT30P
- added P7: XT90PW-M, precharge:XT90PW-M
- added Q3: TPH1R204PL, imu_junction:TPH1R204PL
- added R10: 220, mfpassives:RESISTOR_0603
- added U6: TCAN334G, precharge:TCAN334G
- C3: value 2.2uF -> 0.1uF; device mfpassives:CAPACITOR_NP_0603 -> mfpassives:CAPACITOR_NP_0402; HOUSEPART (none) -> 1; MF KEMET -> (none); MPN C0603C225K8PACTU -> MF-CAP-0402-0.1uF
- C4, C5, C6: device mfpassives:CAPACITOR_NP_0603 -> mfpassives:CAPACITOR_NP_0402; MPN MF-CAP-0603-0.1uF -> MF-CAP-0402-0.1uF
- U$1, U$2, U$3, U$4: value MOUNTM2 -> MOUNT; device controller:MOUNTM2 -> precharge:MOUNT
- U2: value LP2985SOT-23-5 -> MAX150628TDFN; device precharge:LP2985SOT-23-5 -> precharge:MAX150628TDFN; MF TI -> (none); MPN LP2985IM5X-3.3/NOPB -> (none); POPULATE 1 -> (none)
- U3: value ATTINY44A-SSU -> STM32G474CEU6; device absolute_position:ATTINY44A-SSU -> precharge:STM32G474CEU6; MF MICROCHIP -> (none); MPN ATTINY44ASSU -> (none); POPULATE 1 -> (none)
Connections:
- removed net MISO: JP1.1, U3.PA5
- removed net MOSI: JP1.4, U3.PA6
- removed net N$5: D2.CATHODE, U3.PA3
- removed net RST: JP1.5, U3.PB3
- removed net SCK: JP1.3, U3.PA4
- new net CAN_N: CAN1.2, CAN2.2, U6.CANL
- new net CAN_P: CAN1.1, CAN2.1, U6.CANH
- new net CAN_RX: U3.PA11, U6.RXD
- new net CAN_SHDN: U3.PA10, U6.SHDN
- new net CAN_TX: U3.PA12, U6.TXD
- new net LED1: D1.CATHODE, U3.PC15-OSC32_OUT
- new net LED2: D2.CATHODE, U3.PC14-OSC32_IN
- new net LX: L1.P$1, U2.LX
- new net N$13: C9.P$1, U2.VCC
- new net NRST: C3.P$1, J1.2, U3.PG10-NRST
- new net PWR_LED: J2.2, U3.PA2
- new net PWR_SW: J2.3, U3.PA3
- new net SWCLK: J1.5, U3.PA14
- new net SWDIO: J1.3, U3.PA13
- net +12V: now also D12.P$1; no longer U2.EN, U2.IN
- net +18V: now also C8.P$1, P1.2, P2.2, P3.2, P4.2, P5.2, P6.2, P7.1, U2.EN, U2.VIN; no longer V+.P$1, V+OUT.P$1
- net FET_MAIN: now also U3.PA1; no longer U3.PB0
- net FET_PRECHARGE: now also U3.PA0; no longer U3.PB1
- net GND: now also C10.P$2, C11.P$2, C12.P$2, C13.P$2, C14.P$2, C15.P$2, C7.P$2, C8.P$2, C9.P$2, CAN1.3, CAN2.3, DG.P$1, J1.4, J2.4, P7.2, Q3.S, U3.THERMALPAD, U3.VSSA, U3.VSS_1, U3.VSS_2, U3.VSS_3, U6.GND, U6.STB; no longer JP1.6, U3.GND, V-.P$1
- net N$2: now also J2.1, R10.P$1; no longer D1.CATHODE, U3.PA2
- net N$3: now also Q3.G
- net V-OUT: now also P1.1, P2.1, P3.1, P4.1, P5.1, P6.1, Q3.D; no longer V-OUT.P$1
- net VCC: now also C10.P$1, C11.P$1, C12.P$1, C13.P$1, C14.P$1, C15.P$1, C7.P$1, D3V3.P$1, J1.6, L1.P$2, R10.P$2, U2.FB, U3.VDDA, U3.VDD_1, U3.VDD_2, U3.VDD_3, U3.VREF+, U6.VCC; no longer C3.P$1, JP1.2, U2.OUT, U3.VCC
- net VSAMP_IN: now also U3.PA9; no longer U3.PA0
- net VSAMP_OUT: now also U3.PA8; no longer U3.PA1
Other:
- note added: "CONNECTORS / MOUNTS"
- note added: "CONTROLLER"
- note added: "INTERFACE"
- note added: "POWER"
- note added: "REGULATORS"
- note added: "SENSE / DBG"
- note added: "moteus power dist (c) 2019 Josh Pieper, jjp@pobox.com Licensed under the Apache 2.0 License https://www.apache.org/licenses/LICENSE-2.0"
- note removed: "(c) 2019 Josh Pieper, jjp@pobox.com Licensed under the Apache 2.0 License https://www.apache.org/licenses/LICENSE-2.0"
- moved on the sheet: C1, C2, C3, C4, C5, C6, D1, D2, D3, Q1, Q2, R1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

Commit message: power_dist: All BOM filled in
Parts:
- CAN1, CAN2: MF (none) -> JST; MPN (none) -> B3B-PH-SM4-TB(LF)(SN); POPULATE (none) -> 1
- D12, D3V3, DG, P1, P2, P3, P4, P5, P6, P7: POPULATE (none) -> 0
- J1: MF (none) -> JST; MPN (none) -> B6B-ZR-SM4-TF(LF)(SN); POPULATE (none) -> 1
- J2: MF (none) -> JST; MPN (none) -> B4B-PH-SM4-TB(LF)(SN); POPULATE (none) -> 1
- L1: POPULATE (none) -> 1
- U2: MF (none) -> MAXIM; MPN (none) -> MAX15062AATA+T; POPULATE (none) -> 1
- U3: MF (none) -> ST; MPN (none) -> STM32G474CEU6; POPULATE (none) -> 1
- U6: MF (none) -> TI; MPN (none) -> TCAN334GDCNR; POPULATE (none) -> 1

Commit message: power dist: Fix some silks and MPNs found by macrofab
Parts:
- Q1, Q2, Q3: MPN (none) -> TPH1R204PL,L1Q
- U1: MPN (none) -> ZXTR2012Z-13
Changed lines of the file:
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@@
 <parts>
 <part name="U4" library="imu_junction" deviceset="MIC4416" device=""/>
-<part name="Q1" library="imu_junction" deviceset="TPH1R204PL" device=""/>
+<part name="Q1" library="imu_junction" deviceset="TPH1R204PL" device="">
+<attribute name="MPN" value="TPH1R204PL,L1Q"/>
+</part>
 <part name="R7" library="mfpassives" deviceset="RESISTOR" device="_1206" value="10 1W">
 <attribute name="MF" value="Susumu"/>
@@
 </part>
 <part name="U5" library="imu_junction" deviceset="MIC4416" device=""/>
-<part name="Q2" library="imu_junction" deviceset="TPH1R204PL" device=""/>
+<part name="Q2" library="imu_junction" deviceset="TPH1R204PL" device="">
+<attribute name="MPN" value="TPH1R204PL,L1Q"/>
+</part>
 <part name="GND13" library="supply1" deviceset="GND" device=""/>
 <part name="D1" library="mfleds" deviceset="LED_SINGLE" device="-0603">
@@
 </part>
 <part name="P+2" library="supply1" deviceset="VCC" device=""/>
-<part name="U1" library="imu_junction" deviceset="ZXTR2012Z" device=""/>
+<part name="U1" library="imu_junction" deviceset="ZXTR2012Z" device="">
+<attribute name="MPN" value="ZXTR2012Z-13"/>
+</part>
 <part name="GND9" library="supply1" deviceset="GND" device=""/>
 <part name="P+4" library="supply1" deviceset="+18V" device=""/>
@@
 <attribute name="POPULATE" value="1"/>
 </part>
-<part name="Q3" library="imu_junction" deviceset="TPH1R204PL" device=""/>
+<part name="Q3" library="imu_junction" deviceset="TPH1R204PL" device="">
+<attribute name="MPN" value="TPH1R204PL,L1Q"/>
+</part>
 <part name="GND20" library="supply1" deviceset="GND" device=""/>
 <part name="D12" library="precharge" deviceset="PAD" device="24AWG_PAD">

Commit message: Update TCAN334G MPN to the SOIC variant
It appears that the digikey librarian erroneously labeled the SOIC8
footprint as SOT23-8.
Parts:
- U6: MPN TCAN334GDCNR -> TCAN334GDR
Changed lines of the file:
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@@
 <part name="U6" library="precharge" deviceset="TCAN334G" device="">
 <attribute name="MF" value="TI"/>
-<attribute name="MPN" value="TCAN334GDCNR"/>
+<attribute name="MPN" value="TCAN334GDR"/>
 <attribute name="POPULATE" value="1"/>
 </part>

Commit message: Update power dist board to r2
Parts:
- added DI: PAD24AWG_PAD, precharge:PAD24AWG_PAD
Connections:
- net +18V: now also DI.P$1, P7.2; no longer P7.1
- net GND: now also P7.1; no longer P7.2, U3.VSSA, U3.VSS_1, U3.VSS_2, U3.VSS_3
- net SWCLK: now also U3.PA15; no longer U3.PA14
- net SWDIO: now also U3.PA14; no longer U3.PA13
Changed lines of the file:
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@@
 <part name="P+18" library="supply1" deviceset="VCC" device=""/>
 <part name="P+19" library="supply1" deviceset="+12V" device=""/>
+<part name="DI" library="precharge" deviceset="PAD" device="24AWG_PAD">
+<attribute name="POPULATE" value="0"/>
+</part>
+<part name="P+20" library="supply1" deviceset="+18V" device=""/>
 </parts>
 <sheets>
@@
 <instance part="GND7" gate="1" x="228.6" y="-30.48"/>
 <instance part="GND8" gate="1" x="-30.48" y="127"/>
-<instance part="P+9" gate="1" x="-30.48" y="160.02"/>
+<instance part="P+9" gate="1" x="-38.1" y="160.02"/>
 <instance part="P+10" gate="1" x="-5.08" y="157.48"/>
 <instance part="C5" gate="G$1" x="2.54" y="-5.08"/>
@@
 <instance part="P+18" gate="VCC" x="287.02" y="-17.78"/>
 <instance part="P+19" gate="1" x="287.02" y="-5.08"/>
+<instance part="DI" gate="G$1" x="307.34" y="10.16">
+<attribute name="POPULATE" x="307.34" y="10.16" size="1.778" layer="96" font="vector" display="off"/>
+</instance>
+<instance part="P+20" gate="1" x="284.48" y="17.78"/>
 </instances>
 <busses>
@@
 </segment>
 <segment>
-<pinref part="P7" gate="G$1" pin="2"/>
 <pinref part="GND8" gate="1" pin="GND"/>
-<wire x1="-48.26" y1="137.16" x2="-30.48" y2="137.16" width="0.1524" layer="91"/>
-<wire x1="-30.48" y1="137.16" x2="-30.48" y2="129.54" width="0.1524" layer="91"/>
+<wire x1="-30.48" y1="139.7" x2="-30.48" y2="129.54" width="0.1524" layer="91"/>
+<pinref part="P7" gate="G$1" pin="1"/>
+<wire x1="-48.26" y1="139.7" x2="-30.48" y2="139.7" width="0.1524" layer="91"/>
 </segment>
 <segment>
@@
 <wire x1="454.66" y1="182.88" x2="454.66" y2="175.26" width="0.1524" layer="91"/>
 <junction x="444.5" y="182.88"/>
-<pinref part="U3" gate="G$1" pin="VSS_3"/>
-<wire x1="454.66" y1="182.88" x2="459.74" y2="182.88" width="0.1524" layer="91"/>
-<wire x1="459.74" y1="182.88" x2="459.74" y2="175.26" width="0.1524" layer="91"/>
-<junction x="454.66" y="182.88"/>
-</segment>
-<segment>
-<pinref part="U3" gate="G$1" pin="VSS_2"/>
-<wire x1="492.76" y1="149.86" x2="513.08" y2="149.86" width="0.1524" layer="91"/>
-<wire x1="513.08" y1="149.86" x2="513.08" y2="152.4" width="0.1524" layer="91"/>
+</segment>
+<segment>
 <pinref part="GND17" gate="1" pin="GND"/>
-<wire x1="513.08" y1="152.4" x2="523.24" y2="152.4" width="0.1524" layer="91"/>
 <pinref part="C11" gate="G$1" pin="P$2"/>
 <wire x1="523.24" y1="152.4" x2="523.24" y2="154.94" width="0.1524" layer="91"/>
-<junction x="523.24" y="152.4"/>
 </segment>
 <segment>
@@
 <wire x1="459.74" y1="83.82" x2="469.9" y2="83.82" width="0.1524" layer="91"/>
 <wire x1="469.9" y1="83.82" x2="477.52" y2="83.82" width="0.1524" layer="91"/>
-<wire x1="477.52" y1="83.82" x2="480.06" y2="83.82" width="0.1524" layer="91"/>
-<wire x1="480.06" y1="83.82" x2="482.6" y2="83.82" width="0.1524" layer="91"/>
+<wire x1="477.52" y1="83.82" x2="482.6" y2="83.82" width="0.1524" layer="91"/>
 <wire x1="482.6" y1="83.82" x2="497.84" y2="83.82" width="0.1524" layer="91"/>
 <wire x1="497.84" y1="83.82" x2="497.84" y2="86.36" width="0.1524" layer="91"/>
@@
 <wire x1="477.52" y1="83.82" x2="477.52" y2="81.28" width="0.1524" layer="91"/>
 <junction x="477.52" y="83.82"/>
-<pinref part="U3" gate="G$1" pin="VSS_1"/>
-<wire x1="480.06" y1="106.68" x2="480.06" y2="96.52" width="0.1524" layer="91"/>
-<junction x="480.06" y="83.82"/>
-<pinref part="U3" gate="G$1" pin="VSSA"/>
-<wire x1="480.06" y1="96.52" x2="480.06" y2="83.82" width="0.1524" layer="91"/>
-<wire x1="469.9" y1="106.68" x2="469.9" y2="96.52" width="0.1524" layer="91"/>
-<wire x1="469.9" y1="96.52" x2="480.06" y2="96.52" width="0.1524" layer="91"/>
-<junction x="480.06" y="96.52"/>
 </segment>
 <segment>
@@
 </segment>
 <segment>
-<pinref part="U3" gate="G$1" pin="VDD_2"/>
-<wire x1="492.76" y1="152.4" x2="508" y2="152.4" width="0.1524" layer="91"/>
-<wire x1="508" y1="152.4" x2="508" y2="160.02" width="0.1524" layer="91"/>
+<wire x1="508" y1="149.86" x2="508" y2="160.02" width="0.1524" layer="91"/>
 <pinref part="C11" gate="G$1" pin="P$1"/>
 <wire x1="508" y1="160.02" x2="523.24" y2="160.02" width="0.1524" layer="91"/>
@@
 <wire x1="523.24" y1="160.02" x2="523.24" y2="165.1" width="0.1524" layer="91"/>
 <junction x="523.24" y="160.02"/>
+<pinref part="U3" gate="G$1" pin="VDD_2"/>
+<wire x1="492.76" y1="149.86" x2="508" y2="149.86" width="0.1524" layer="91"/>
 </segment>
 <segment>
@@
 <wire x1="469.9" y1="93.98" x2="472.44" y2="93.98" width="0.1524" layer="91"/>
 <wire x1="472.44" y1="93.98" x2="474.98" y2="93.98" width="0.1524" layer="91"/>
-<wire x1="474.98" y1="93.98" x2="482.6" y2="93.98" width="0.1524" layer="91"/>
+<wire x1="474.98" y1="93.98" x2="480.06" y2="93.98" width="0.1524" layer="91"/>
+<wire x1="480.06" y1="93.98" x2="482.6" y2="93.98" width="0.1524" layer="91"/>
 <wire x1="482.6" y1="93.98" x2="495.3" y2="93.98" width="0.1524" layer="91"/>
 <wire x1="495.3" y1="93.98" x2="497.84" y2="93.98" width="0.1524" layer="91"/>
@@
 <wire x1="495.3" y1="109.22" x2="495.3" y2="93.98" width="0.1524" layer="91"/>
 <junction x="495.3" y="93.98"/>
-<pinref part="U3" gate="G$1" pin="VDD_1"/>
-<wire x1="482.6" y1="106.68" x2="482.6" y2="93.98" width="0.1524" layer="91"/>
 <pinref part="U3" gate="G$1" pin="VDDA"/>
 <wire x1="474.98" y1="106.68" x2="474.98" y2="93.98" width="0.1524" layer="91"/>
@@
 <wire x1="472.44" y1="106.68" x2="472.44" y2="93.98" width="0.1524" layer="91"/>
 <junction x="472.44" y="93.98"/>
+<pinref part="U3" gate="G$1" pin="VDD_1"/>
+<wire x1="480.06" y1="106.68" x2="480.06" y2="93.98" width="0.1524" layer="91"/>
+<junction x="480.06" y="93.98"/>
 </segment>
 <segment>
@@
 <segment>
 <pinref part="P+9" gate="1" pin="+18V"/>
-<pinref part="P7" gate="G$1" pin="1"/>
-<wire x1="-48.26" y1="139.7" x2="-30.48" y2="139.7" width="0.1524" layer="91"/>
-<wire x1="-30.48" y1="139.7" x2="-30.48" y2="157.48" width="0.1524" layer="91"/>
+<wire x1="-38.1" y1="137.16" x2="-38.1" y2="157.48" width="0.1524" layer="91"/>
+<pinref part="P7" gate="G$1" pin="2"/>
+<wire x1="-38.1" y1="137.16" x2="-48.26" y2="137.16" width="0.1524" layer="91"/>
 </segment>
 <segment>
@@
 <junction x="60.96" y="139.7"/>
 </segment>
+<segment>
+<pinref part="P+20" gate="1" pin="+18V"/>
+<wire x1="284.48" y1="15.24" x2="284.48" y2="10.16" width="0.1524" layer="91"/>
+<pinref part="DI" gate="G$1" pin="P$1"/>
+<wire x1="284.48" y1="10.16" x2="299.72" y2="10.16" width="0.1524" layer="91"/>
+</segment>
 </net>
 <net name="+12V" class="1">
@@
 </segment>
 <segment>
-<pinref part="U3" gate="G$1" pin="PA13"/>
+<pinref part="U3" gate="G$1" pin="PA14"/>
 <wire x1="485.14" y1="175.26" x2="485.14" y2="203.2" width="0.1524" layer="91"/>
 <label x="485.14" y="198.12" size="1.778" layer="95" font="vector" rot="R90"/>
@@
 </segment>
 <segment>
-<pinref part="U3" gate="G$1" pin="PA14"/>
+<pinref part="U3" gate="G$1" pin="PA15"/>
 <wire x1="482.6" y1="175.26" x2="482.6" y2="203.2" width="0.1524" layer="91"/>
 <label x="482.6" y="198.12" size="1.778" layer="95" font="vector" rot="R90"/>

Commit message: More power dist errata:
 * Fix 10k resistors
 * Rename TCAN package to actually be SOIC8, since that is what it is
Parts:
- R4, R6: MPN ERT-J1VG103FA -> P10.0KHDKR-ND
Changed lines of the file:
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@@
 <part name="R4" library="mfpassives" deviceset="RESISTOR" device="_0603" value="10k 1%">
 <attribute name="MF" value="PANASONIC"/>
-<attribute name="MPN" value="ERT-J1VG103FA"/>
+<attribute name="MPN" value="P10.0KHDKR-ND"/>
 </part>
 <part name="R5" library="mfpassives" deviceset="RESISTOR" device="_0603" value="100k 1%">
@@
 <part name="R6" library="mfpassives" deviceset="RESISTOR" device="_0603" value="10k 1%">
 <attribute name="MF" value="PANASONIC"/>
-<attribute name="MPN" value="ERT-J1VG103FA"/>
+<attribute name="MPN" value="P10.0KHDKR-ND"/>
 </part>
 <part name="P+8" library="supply1" deviceset="+18V" device=""/>

Commit message: Use MPNs instead of digikey part numbers
Parts:
- R4, R6: MPN P10.0KHDKR-ND -> ERJ-3EKF1002V
Changed lines of the file:
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@@
 <part name="R4" library="mfpassives" deviceset="RESISTOR" device="_0603" value="10k 1%">
 <attribute name="MF" value="PANASONIC"/>
-<attribute name="MPN" value="P10.0KHDKR-ND"/>
+<attribute name="MPN" value="ERJ-3EKF1002V"/>
 </part>
 <part name="R5" library="mfpassives" deviceset="RESISTOR" device="_0603" value="100k 1%">
@@
 <part name="R6" library="mfpassives" deviceset="RESISTOR" device="_0603" value="10k 1%">
 <attribute name="MF" value="PANASONIC"/>
-<attribute name="MPN" value="P10.0KHDKR-ND"/>
+<attribute name="MPN" value="ERJ-3EKF1002V"/>
 </part>
 <part name="P+8" library="supply1" deviceset="+18V" device=""/>
